File: Board1/Board1.kicad_sch (KiCad schematic)
At the start: 0 parts

Commit message: v1.2 release of board with bug fixes etc
Other:
- sheet Power - 240AC to 5VDC renamed Power - 240VAC to 5VDC
- removed sheet IO - Thermocouple
- note added: "Page2"
- note added: "Page3"
- note added: "Page4"
- note added: "Page5"
- note added: "Page6"
- note added: "Page7"
- note added: "Page8"
- note removed: "TOP VIEW"
