File: Board1/sch_pcb_mounts.kicad_sch (KiCad schematic)
At the start: 4 parts

Commit message: v1.2 release of board with bug fixes etc
Changed lines of the file:
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@@
 (kicad_sch
-	(version 20231120)
+	(version 20250114)
 	(generator "eeschema")
-	(generator_version "8.0")
+	(generator_version "9.0")
 	(paper "A4")
 	(title_block
 		(title "Mounting Holes")
-		(date "2025-02-19")
-		(rev "1.1")
+		(date "2025-03-08")
+		(rev "1.2")
 		(company "Wattle Labs")
 	)
@@
 		(at 12.065 12.065 0)
 		(size 273.05 13.335)
+		(margins 2.2499 2.2499 2.2499 2.2499)
 		(stroke
 			(width -0.0001)
